Commit message: fix: 第一版新雷达代码

File: ros2_ws/src/alohamini_description/urdf/alohamini_nav.urdf (robot description, URDF)
Before this commit: robot Aloha, 21 links, 20 joints
Links:
- removed link imu_frame
Joints:
- removed joint base_link_to_imu_frame
- joint base_link_to_laser_frame: origin xyz=0 -0.20 0.12 rpy=0 0 0 -> xyz=0 -0.20 0.12 rpy=0 0 1.5707963267948966
